Commit message: Change wheel collision from cylinder to sphere

File: description/robot_core.xacro (robot description, xacro)
@@ -63,5 +63,6 @@
         <collision>
             <geometry>
-                <cylinder radius="0.05" length="0.04"/>
+                <!-- <cylinder radius="0.05" length="0.04"/> -->
+                <sphere radius="0.05"/>
             </geometry>
             <material name="blue"/>
@@ -92,5 +93,6 @@
         <collision>
             <geometry>
-                <cylinder radius="0.05" length="0.04"/>
+                <!-- <cylinder radius="0.05" length="0.04"/> -->
+                <sphere radius="0.05"/>
             </geometry>
             <material name="blue"/>
